Commit message: images

File: src/robot_description/src/description/robot.urdf (robot description, URDF)
Before this commit: robot diff_drive_robot, 8 links, 7 joints
Joints:
- joint left_wheel_joint: limit lower=-333.14 upper=333.14 effort=100 velocity=10 -> lower=-1000 upper=1000 effort=100 velocity=10
- joint right_wheel_joint: limit lower=-333.14 upper=333.14 effort=100 velocity=10 -> lower=-1000 upper=1000 effort=100 velocity=10
